File: _autosave-PDArcadeSliderPCB.sch (KiCad schematic (older format))
At the start: 17 parts, among them J1 Conn_01x01_Male, J10 topgroundhatching, J2 Conn_01x06_Male, J3 Conn_01x01, J4 Conn_01x01, J5 Conn_01x01_Male, J6 Conn_01x01_Male, J7 Conn_01x01_Male, J8 Conn_01x01_Male, J9 Conn_01x01_Male, U1 testsensorg, U2 testsensorg, U3 testsensorg, U4 testsensorg, U5 testsensorg, U6 testsensorg

Commit message: Ground hatching from old manual
Ground hatching from old manual
https://forum.kicad.info/t/copper-pour-with-hatched-fill-instead-of-solid-fill/860/8
because for now KiCad cannot make hatching like this
Parts:
- J11: renamed from J?; footprint PDArcadeSliderPCB:TopHatching -> PDArcadeSliderPCB:bottomhatching
Changed lines of the file:
@@
 	7650 4300 7650 4750
 $Comp
-L PDArcadeSliderPCBsensorlib:topgroundhatching J?
+L PDArcadeSliderPCBsensorlib:topgroundhatching J11
 U 1 1 5DF747A8
 P 8900 4700
-F 0 "J?" H 8980 4742 50  0000 L CNN
+F 0 "J11" H 8980 4742 50  0000 L CNN
 F 1 "topgroundhatching" H 8980 4651 50  0000 L CNN
-F 2 "PDArcadeSliderPCB:TopHatching" H 8900 4700 50  0001 C CNN
+F 2 "PDArcadeSliderPCB:bottomhatching" H 8900 4700 50  0001 C CNN
 F 3 "~" H 8900 4700 50  0001 C CNN
 	1    8900 4700
